Commit message: updated launch files

File: simulation_ws/src/robot_description/urdf/robot.xacro (robot description, xacro)
@@ -1,20 +1,19 @@
 <?xml version="1.0" ?>
-<robot name="robot" xmlns:xacro="https://www.ros.org/wiki/xacro" >
+<robot name="varad_bot" xmlns:xacro="https://www.ros.org/wiki/xacro">
   <!-- Include the Xacro files -->
   <xacro:include filename="$(find robot_description)/urdf/materials.xacro" />
   <xacro:include filename="$(find robot_description)/urdf/gazebo.xacro" />
   <xacro:include filename="$(find robot_description)/urdf/macro.xacro" />
-  <!-- chassis definition -->
+  <!-- Base Chassis -->
   <link name="link_chassis">
-    <!-- pose and inertial -->
     <pose>0 0 0.1 0 0 0</pose>
     <inertial>
       <mass value="5"/>
       <origin rpy="0 0 0" xyz="0 0 0.1"/>
-      <inertia ixx="0.0395416666667" ixy="0" ixz="0" iyy="0.106208333333" iyz="0" izz="0.106208333333"/>
+      <inertia ixx="0.04" ixy="0" ixz="0" iyy="0.04" iyz="0" izz="0.04"/>
     </inertial>
     <collision name="collision_chassis">
       <geometry>
-        <cylinder length="0.05" radius="0.3"/>
+        <box size="0.5 0.3 0.1"/>
       </geometry>
     </collision>
@@ -22,68 +21,26 @@
       <origin rpy="0 0 0" xyz="0 0 0"/>
       <geometry>
-        <cylinder length="0.05" radius="0.3"/>
+        <box size="0.5 0.3 0.1"/>
       </geometry>
-      <material name="blue"/>
-    </visual>
-    <!-- caster front -->
-    <collision name="caster_front_collision">
-      <origin rpy=" 0 0 0" xyz="0.35 0 -0.05"/>
-      <geometry>
-        <sphere radius="0.05"/>
-      </geometry>
-      <surface>
-        <friction>
-          <ode>
-            <mu>0</mu>
-            <mu2>0</mu2>
-            <slip1>1.0</slip1>
-            <slip2>1.0</slip2>
-          </ode>
-        </friction>
-      </surface>
-    </collision>
-    <visual name="caster_front_visual">
-      <origin rpy=" 0 0 0" xyz="0.2 0 -0.05"/>
-      <geometry>
-        <sphere radius="0.05"/>
-      </geometry>
+      <material name="red"/>
     </visual>
   </link>
-  <!-- Link for laser -->
-  <link name="sensor_laser">
-    <inertial>
-      <origin xyz="0 0 0" rpy="0 0 0" />
-      <mass value="4" />
-      <xacro:cylinder_inertia mass="1" r="0.05" l="0.1" />
-    </inertial>
-    <visual>
-      <origin xyz="0 0 0" rpy="0 0 0" />
-      <geometry>
-        <cylinder radius="0.05" length="0.1"/>
-      </geometry>
-      <material name="white" />
-      <material name="laserLight" />
-    </visual>
-    <collision>
-      <origin xyz="0 0 0" rpy="0 0 0"/>
-      <geometry>
-        <cylinder radius="0.05" length="0.1"/>
-      </geometry>
-      <material name="collisionLaser" />
-    </collision>
-  </link>
-  <!-- Joint for laser -->
-  <joint name="joint_sensor_laser" type="fixed">
-    <origin xyz="0.15 0 0.05" rpy="0 0 0"/>
-    <parent link="link_chassis"/>
-    <child link="sensor_laser"/>
-  </joint>
-  <!-- Right Wheel Link -->
-  <xacro:link_wheel name="link_right_wheel" />
-  <!--   Joint for right wheel  -->
-  <xacro:joint_wheel name="joint_right_wheel"  child="link_right_wheel"  origin_xyz="-0.05 0.3 0"  />
-  <!-- Left Wheel link -->
-  <xacro:link_wheel name="link_left_wheel" />
-  <!--   Joint for left wheel  -->
-  <xacro:joint_wheel name="joint_left_wheel"   child="link_left_wheel"   origin_xyz="-0.05 -0.3 0"  />
-</robot>
+  <!-- Front caster -->
+  <collision name="caster_front_collision">
+    <origin rpy="0 0 0" xyz="0.35 0 -0.05"/>
+    <geometry>
+      <box size="0.5 0.5 0.1"/>
+    </geometry>
+    <surface>
+      <friction>
+        <ode>
+          <mu>0</mu>
+          <mu2>0</mu2>
+          <slip1>1.0</slip1>
+          <slip2>1.0</slip2>
+        </ode>
+      </friction>
+    </surface>
+  </collision>
+  <visual name="caster_front_visual">
+    <origin rpy="0 0 0" xyz="0.2 0 -0.0
